Commit message: wip description

File: slammer_description/urdf/m2wr.xacro (robot description, xacro)
@@ -5,9 +5,10 @@
   <xacro:include filename="$(find unav2_hardware)/urdf/macros.xacro" />
   <link name="link_chassis">
+    <parent link="base_link"/>
     <!-- pose and inertial -->
-    <pose>0 0 0.1 0 0 0</pose>
+    <pose>0 0 0 0 0 0</pose>
     <inertial>
       <mass value="5"/>
-      <origin rpy="0 0 0" xyz="0 0 0.1"/>
+      <origin rpy="0 0 0" xyz="0 0 0.075"/>
       <inertia ixx="0.0395416666667" ixy="0" ixz="0" iyy="0.106208333333" iyz="0" izz="0.106208333333"/>
     </inertial>
@@ -15,5 +16,5 @@
     <collision name="collision_chassis">
       <geometry>
-        <box size="0.5 0.3 0.07"/>
+        <box size="0.36 0.30 0.07"/>
       </geometry>
     </collision>
@@ -21,31 +22,9 @@
       <origin rpy="0 0 0" xyz="0 0 0"/>
       <geometry>
-        <box size="0.5 0.3 0.07"/>
+        <box size="0.36 0.30 0.07"/>
       </geometry>
       <material name="blue"/>
     </visual>
     <!-- caster front -->
-    <collision name="caster_front_collision">
-      <origin rpy=" 0 0 0" xyz="0.35 0 -0.05"/>
-      <geometry>
-        <sphere radius="0.05"/>
-      </geometry>
-      <surface>
-        <friction>
-          <ode>
-            <mu>0</mu>
-            <mu2>0</mu2>
-            <slip1>1.0</slip1>
-            <slip2>1.0</slip2>
-          </ode>
-        </friction>
-      </surface>
-    </collision>
-    <visual name="caster_front_visual">
-      <origin rpy=" 0 0 0" xyz="0.2 0 -0.05"/>
-      <geometry>
-        <sphere radius="0.05"/>
-      </geometry>
-    </visual>
   </link>
   <link name="sensor_laser">
@@ -75,5 +54,5 @@
   </joint>
   <xacro:link_wheel name="link_right_wheel" />
-  <xacro:joint_wheel name="joint1" child="link_right_wheel" origin_xyz="-0.05 0.20 0" />
+  <xacro:joint_wheel name="joint1" child="link_right_wheel" origin_xyz="-0.05 0.40 0" />
   <xacro:link_wheel name="link_left_wheel" />
   <xacro:joint_wheel name="joint2" child="link_left_wheel" origin_xyz="-0.05 -0.20 0" />

Commit message: Fix and cleanup description/urdf

File: slammer_description/urdf/m2wr.xacro (robot description, xacro)
@@ -1,11 +1,55 @@
 <?xml version="1.0" ?>
-<robot name="m2wr" xmlns:xacro="http://www.ros.org/wiki/xacro">
-  <xacro:include filename="$(find unav2_hardware)/urdf/materials.xacro" />
-  <xacro:include filename="$(find unav2_hardware)/urdf/m2wr.gazebo" />
-  <xacro:include filename="$(find unav2_hardware)/urdf/macros.xacro" />
+<robot name="m2wr"
+  xmlns:xacro="http://www.ros.org/wiki/xacro">
+  <xacro:property name="body_lenght" value="0.30"/>
+  <xacro:property name="body_width" value="0.16"/>
+  <xacro:property name="body_height" value="0.055"/>
+  <xacro:property name="body_ground_clearance" value="0.082"/>
+  <xacro:property name="total_lenght" value="0.30"/>
+  <xacro:property name="total_width" value="0.30"/>
+  <xacro:property name="total_height" value="0.20"/>
+  <xacro:property name="laser_x_displacement" value="0.04"/>
+  <xacro:property name="laser_z_displacement" value="0.095"/>
+  <xacro:property name="laser_height" value="0.055"/>
+  <xacro:property name="laser_radius" value="0.035"/>
+  <xacro:property name="wheel_front_x_displacement" value="0.09"/>
+  <xacro:property name="wheel_rear_x_displacement" value="-0.09"/>
+  <xacro:property name="wheel_y_displacement" value="0.12"/>
+  <xacro:property name="wheel_z_displacement" value="-0.02"/>
+  <xacro:property name="imu_x_displacement" value="-0.08"/>
+  <xacro:property name="imu_y_displacement" value="-0.05"/>
+  <xacro:property name="imu_z_displacement" value="0.055"/>
+  <xacro:property name="imu_rpy" value="${pi} 0.0 0.0"/>
+  <xacro:property name="camera_x_displacement" value="0.145"/>
+  <xacro:property name="camera_y_displacement" value="0.0"/>
+  <xacro:property name="camera_z_displacement" value="0.07"/>
+  <xacro:property name="camera_rpy" value="0 -0.2 0"/>
+  <xacro:include filename="$(find slammer_description)/urdf/materials.xacro" />
+  <xacro:include filename="$(find slammer_description)/urdf/m2wr.gazebo" />
+  <xacro:include filename="$(find slammer_description)/urdf/macros.xacro" />
+  <!-- base link with global collision geometry -->
+  <link name="base_link">
+    <visual>
+      <origin rpy="0 0 0" xyz="0 0 ${total_height / 2}"/>
+      <geometry>
+        <box size="${total_lenght} ${total_width} ${total_height}"/>
+      </geometry>
+      <material name="invisible_grey"/>
+    </visual>
+    <collision>
+      <origin rpy="0 0 0" xyz="0 0 ${total_height / 2}"/>
+      <geometry>
+        <box size="${total_lenght} ${total_width} ${total_height}"/>
+      </geometry>
+    </collision>
+  </link>
+  <!-- chassis/body -->
+  <joint name="base_link_to_link_chassis" type="fixed">
+    <origin xyz="0 0 ${body_ground_clearance}" rpy="0 0 0"/>
+    <parent link="base_link"/>
+    <child link="link_chassis"/>
+  </joint>
   <link name="link_chassis">
-    <parent link="base_link"/>
     <!-- pose and inertial -->
-    <pose>0 0 0 0 0 0</pose>
     <inertial>
       <mass value="5"/>
@@ -16,17 +60,23 @@
     <collision name="collision_chassis">
       <geometry>
-        <box size="0.36 0.30 0.07"/>
+        <box size="${body_lenght} ${body_width} ${body_height}"/>
       </geometry>
     </collision>
     <visual>
-      <origin rpy="0 0 0" xyz="0 0 0"/>
+      <origin rpy="0 0 0" xyz="0 0 ${body_height / 2}"/>
       <geometry>
-        <box size="0.36 0.30 0.07"/>
+        <box size="${body_lenght} ${body_width} ${body_height}"/>
       </geometry>
-      <material name="blue"/>
+      <material name="transp_white"/>
     </visual>
     <!-- caster front -->
   </link>
-  <link name="sensor_laser">
+  <!-- Lidar -->
+  <joint name="link_chassis_to_laser" type="fixed">
+    <origin xyz="${laser_x_displacement} 0 ${laser_z_displacement}" rpy="0 0 0"/>
+    <parent link="link_chassis"/>
+    <child link="laser"/>
+  </joint>
+  <link name="laser">
     <inertial>
       <origin xyz="0 0 0" rpy="0 0 0" />
@@ -35,25 +85,74 @@
     </inertial>
     <visual>
-      <origin xyz="0 0 0" rpy="0 0 0" />
+      <origin xyz="0 0 ${- laser_z_displacement + body_height + laser_height / 2}" rpy="0 0 0" />
       <geometry>
-        <cylinder radius="0.05" length="0.1"/>
+        <cylinder radius="${laser_radius}" length="${laser_height}"/>
       </geometry>
       <material name="white" />
     </visual>
     <collision>
-      <origin xyz="0 0 0" rpy="0 0 0"/>
+      <origin xyz="0 0 ${- laser_z_displacement + body_height + laser_height / 2}" rpy="0 0 0" />
       <geometry>
-        <cylinder radius="0.05" length="0.1"/>
+        <cylinder radius="${laser_radius}" length="${laser_height}"/>
       </geometry>
     </collision>
   </link>
-  <joint name="joint_sensor_laser" type="fixed">
-    <origin xyz="0.15 0 0.05" rpy="0 0 0"/>
+  <!-- Wheels -->
+  <xacro:link_wheel name="link_right_wheel" />
+  <xacro:joint_wheel name="joint1" child="link_right_wheel" origin_xyz="${wheel_front_x_displacement} ${wheel_y_displacement} ${wheel_z_displacement}" />
+  <xacro:link_wheel name="link_left_wheel" />
+  <xacro:joint_wheel name="joint2" child="link_left_wheel" origin_xyz="${wheel_front_x_displacement} ${-wheel_y_displacement} ${wheel_z_displacement}" />
+  <xacro:link_wheel name="link_rear_right_wheel" />
+  <xacro:joint_static_wheel name="joint3" child="link_rear_right_wheel" origin_xyz="${wheel_rear_x_displacement} ${wheel_y_displacement} ${wheel_z_displacement}" />
+  <xacro:link_wheel name="link_rear_left_wheel" />
+  <xacro:joint_static_wheel name="joint4" child="link_rear_left_wheel" origin_xyz="${wheel_rear_x_displacement} ${-wheel_y_displacement} ${wheel_z_displacement}" />
+  <!-- IMU -->
+  <joint name="link_chassis_to_imu_bosch" type="fixed">
+    <origin xyz="${imu_x_displacement} ${imu_y_displacement} ${imu_z_displacement}" rpy="${imu_rpy}"/>
     <parent link="link_chassis"/>
-    <child link="sensor_laser"/>
+    <child link="imu_bosch_link"/>
   </joint>
-  <xacro:link_wheel name="link_right_wheel" />
-  <xacro:joint_wheel name="joint1" child="link_right_wheel" origin_xyz="-0.05 0.40 0" />
-  <xacro:link_wheel name="link_left_wheel" />
-  <xacro:joint_wheel name="joint2" child="link_left_wheel" origin_xyz="-0.05 -0.20 0" />
+  <link name="imu_bosch_link">
+    <visual>
+      <origin xyz="0 0 0" rpy="0 0 0"/>
+      <geometry>
+        <cylinder radius="0.001" length="0.005"/>
+      </geometry>
+      <material name="red" />
+    </visual>
+    <visual>
+      <origin xyz="0.01 0 0" rpy="0 0 0"/>
+      <geometry>
+        <box size="0.02 0.001 0.001"/>
+      </geometry>
+      <material name="blue" />
+    </visual>
+  </link>
+  <!-- Camera -->
+  <joint name="link_chassis_to_camera_mount" type="fixed">
+    <origin xyz="${camera_x_displacement} ${camera_y_displacement} ${camera_z_displacement}" rpy="${camera_rpy}"/>
+    <parent link="link_chassis"/>
+    <child link="camera_mount"/>
+  </joint>
+  <link name="camera_mount"/>
+  <joint name="camera_mount_to_camera_link" type="fixed">
+    <origin xyz="0 0.0 0.0" rpy="0 0 0"/>
+    <parent link="camera_mount"/>
+    <child link="camera_link"/>
+  </joint>
+  <link name="camera_link">
+    <visual>
+      <origin xyz="0 0 0" rpy="0 0 0"/>
+      <geometry>
+        <box size="0.01 0.130 0.02"/>
+      </geometry>
+      <material name="blue" />
+    </visual>
+    <collision>
+      <origin xyz="0 0 0" rpy="0 0 0"/>
+      <geometry>
+        <box size="0.01 0.130 0.02"/>
+      </geometry>
+    </collision>
+  </link>
 </robot>

File: slammer_description/urdf/macros.xacro (robot description, xacro)
@@ -1,39 +1,48 @@
 <?xml version="1.0"?>
 <robot xmlns:xacro="http://www.ros.org/wiki/xacro">
-    <xacro:macro name="link_wheel" params="name">
-        <link name="${name}">
-            <inertial>
-              <mass value="0.2"/>
-              <origin rpy="0 1.5707 1.5707" xyz="0 0 0"/>
-              <inertia ixx="0.000526666666667" ixy="0" ixz="0" iyy="0.000526666666667" iyz="0" izz="0.001"/>
-            </inertial>
-            <collision name="link_right_wheel_collision">
-              <origin rpy="0 1.5707 1.5707" xyz="0 0 0"/>
-              <geometry>
-                <cylinder length="0.04" radius="0.1"/>
-              </geometry>
-            </collision>
-            <visual name="${name}_visual">
-              <origin rpy="0 1.5707 1.5707" xyz="0 0 0"/>
-              <geometry>
-                <cylinder length="0.04" radius="0.1"/>
-              </geometry>
-            </visual>
-        </link>
-    </xacro:macro>
-    <xacro:macro name="joint_wheel" params="name child origin_xyz">
-      <joint name="${name}" type="continuous">
-        <origin rpy="0 0 0" xyz="${origin_xyz}"/>
-        <child link="${child}"/>
-        <parent link="link_chassis"/>
-        <axis rpy="0 0 0" xyz="0 1 0"/>
-        <limit effort="10000" velocity="1000"/>
-        <joint_properties damping="1.0" friction="1.0"/>
-      </joint>
-    </xacro:macro>
-    <xacro:macro name="cylinder_inertia" params="mass r l">
-      <inertia  ixx="${mass*(3*r*r+l*l)/12}" ixy = "0" ixz = "0"
-                iyy="${mass*(3*r*r+l*l)/12}" iyz = "0"
-                izz="${mass*(r*r)/2}" />
-    </xacro:macro>
+  <xacro:macro name="link_wheel" params="name">
+    <link name="${name}">
+      <inertial>
+        <mass value="0.2"/>
+        <origin rpy="0 1.5707 1.5707" xyz="0 0 0"/>
+        <inertia ixx="0.000526666666667" ixy="0" ixz="0" iyy="0.000526666666667" iyz="0" izz="0.001"/>
+      </inertial>
+      <collision name="${name}_collision">
+        <origin rpy="0 1.5707 1.5707" xyz="0 0 0"/>
+        <geometry>
+          <cylinder length="0.065" radius="0.06"/>
+        </geometry>
+      </collision>
+      <visual name="${name}_visual">
+        <origin rpy="0 1.5707 1.5707" xyz="0 0 0"/>
+        <geometry>
+          <cylinder length="0.065" radius="0.06"/>
+        </geometry>
+        <material name="black" />
+      </visual>
+    </link>
+  </xacro:macro>
+  <xacro:macro name="joint_static_wheel" params="name child origin_xyz">
+    <joint name="${name}" type="fixed">
+      <origin rpy="0 0 0" xyz="${origin_xyz}"/>
+      <child link="${child}"/>
+      <parent link="link_chassis"/>
+      <!-- <axis rpy="0 0 0" xyz="0 1 0"/>
+      <limit effort="10000" velocity="1000"/>
+      <joint_properties damping="1.0" friction="1.0"/ -->
+    </joint>
+  </xacro:macro>
+  <xacro:macro name="joint_wheel" params="name child origin_xyz">
+    <joint name="${name}" type="fixed">
+      <origin rpy="0 0 0" xyz="${origin_xyz}"/>
+      <child link="${child}"/>
+      <parent link="link_chassis"/>
+      <axis rpy="0 0 0" xyz="0 1 0"/>
+      <limit effort="10000" velocity="1000"/>
+      <joint_properties damping="1.0" friction="1.0"/>
+    </joint>
+  </xacro:macro>
+  <xacro:macro name="cylinder_inertia" params="mass r l">
+    <inertia ixx="${mass*(3*r*r+l*l)/12}" ixy = "0" ixz = "0" iyy="${mass*(3*r*r+l*l)/12}" iyz = "0" izz="${mass*(r*r)/2}" />
+  </xacro:macro>
 </robot>

File: slammer_description/urdf/materials.xacro (robot description, xacro)
@@ -5,11 +5,14 @@
   </material>
   <material name="blue">
-    <color rgba="0.203125 0.23828125 0.28515625 1.0"/>
+    <color rgba="0.1 0.2 0.4 1.0"/>
   </material>
   <material name="green">
     <color rgba="0.0 0.8 0.0 1.0"/>
   </material>
+  <material name="transp_grey">
+    <color rgba="0.2 0.2 0.2 0.8"/>
+  </material>
   <material name="grey">
-    <color rgba="0.2 0.2 0.2 1.0"/>
+    <color rgba="0.2 0.2 0.2 1"/>
   </material>
   <material name="orange">
@@ -25,3 +28,9 @@
     <color rgba="1.0 1.0 1.0 1.0"/>
   </material>
+  <material name="transp_white">
+    <color rgba="1.0 1.0 1.0 0.8"/>
+  </material>
+  <material name="invisible_grey">
+    <color rgba="0.2 0.2 0.2 0.3"/>
+  </material>
 </robot>

Commit message: add rplidar model

File: slammer_description/urdf/m2wr.xacro (robot description, xacro)
@@ -11,6 +11,9 @@
   <xacro:property name="laser_x_displacement" value="0.04"/>
   <xacro:property name="laser_z_displacement" value="0.095"/>
+  <xacro:property name="laser_radius" value="0.035"/>
   <xacro:property name="laser_height" value="0.055"/>
-  <xacro:property name="laser_radius" value="0.035"/>
+  <xacro:property name="laser_model_x_disp" value="0.070"/>
+  <xacro:property name="laser_model_y_disp" value="-0.013"/>
+  <xacro:property name="laser_model_z_disp" value="0.032"/>
   <xacro:property name="wheel_front_x_displacement" value="0.09"/>
   <xacro:property name="wheel_rear_x_displacement" value="-0.09"/>
@@ -85,9 +88,9 @@
     </inertial>
     <visual>
-      <origin xyz="0 0 ${- laser_z_displacement + body_height + laser_height / 2}" rpy="0 0 0" />
+      <origin xyz="${-laser_model_x_disp} ${-laser_model_y_disp} ${-laser_model_z_disp}" rpy="${pi/2} 0 ${pi}" />
       <geometry>
-        <cylinder radius="${laser_radius}" length="${laser_height}"/>
+        <mesh filename="package://slammer_description/meshes/sensors/rplidar.stl" scale="0.001 0.001 0.001"/>
       </geometry>
-      <material name="white" />
+      <material name="black" />
     </visual>
     <collision>

Commit message: [DESCRIPTION] Fix imu orientation

File: slammer_description/urdf/m2wr.xacro (robot description, xacro)
@@ -23,5 +23,5 @@
   <xacro:property name="imu_y_displacement" value="-0.05"/>
   <xacro:property name="imu_z_displacement" value="0.055"/>
-  <xacro:property name="imu_rpy" value="${pi} 0.0 0.0"/>
+  <xacro:property name="imu_rpy" value="0.0 0.0 0.0"/>
   <xacro:property name="camera_x_displacement" value="0.145"/>
   <xacro:property name="camera_y_displacement" value="0.0"/>
@@ -77,5 +77,5 @@
   <!-- Lidar -->
   <joint name="link_chassis_to_laser" type="fixed">
-    <origin xyz="${laser_x_displacement} 0 ${laser_z_displacement}" rpy="0 0 0"/>
+    <origin xyz="${laser_x_displacement} 0 ${laser_z_displacement}" rpy="0 0 ${pi}"/>
     <parent link="link_chassis"/>
     <child link="laser"/>

Commit message: [DESCRIPTION] - imu rotation

File: slammer_description/urdf/m2wr.xacro (robot description, xacro)
@@ -23,5 +23,5 @@
   <xacro:property name="imu_y_displacement" value="-0.05"/>
   <xacro:property name="imu_z_displacement" value="0.055"/>
-  <xacro:property name="imu_rpy" value="0.0 0.0 0.0"/>
+  <xacro:property name="imu_rpy" value="${pi} 0.0 0.0"/>
   <xacro:property name="camera_x_displacement" value="0.145"/>
   <xacro:property name="camera_y_displacement" value="0.0"/>

Commit message: [DESCRIPTION] - Fix imu orientation and camera inclination

File: slammer_description/urdf/m2wr.xacro (robot description, xacro)
@@ -23,9 +23,9 @@
   <xacro:property name="imu_y_displacement" value="-0.05"/>
   <xacro:property name="imu_z_displacement" value="0.055"/>
-  <xacro:property name="imu_rpy" value="${pi} 0.0 0.0"/>
+  <xacro:property name="imu_rpy" value="0 0.0 ${pi}"/>
   <xacro:property name="camera_x_displacement" value="0.145"/>
   <xacro:property name="camera_y_displacement" value="0.0"/>
   <xacro:property name="camera_z_displacement" value="0.07"/>
-  <xacro:property name="camera_rpy" value="0 -0.2 0"/>
+  <xacro:property name="camera_rpy" value="0 0.22 0"/>
   <xacro:include filename="$(find slammer_description)/urdf/materials.xacro" />
   <xacro:include filename="$(find slammer_description)/urdf/m2wr.gazebo" />

Commit message: [DESCRIPTION] - change to new imu orientation

File: slammer_description/urdf/m2wr.xacro (robot description, xacro)
@@ -23,5 +23,5 @@
   <xacro:property name="imu_y_displacement" value="-0.05"/>
   <xacro:property name="imu_z_displacement" value="0.055"/>
-  <xacro:property name="imu_rpy" value="0 0.0 ${pi}"/>
+  <xacro:property name="imu_rpy" value="${pi} 0.0  ${pi}"/>
   <xacro:property name="camera_x_displacement" value="0.145"/>
   <xacro:property name="camera_y_displacement" value="0.0"/>
@@ -47,4 +47,24 @@
     </collision>
   </link>
+  <link name="base_footprint">
+    <visual>
+      <origin rpy="0 0 0" xyz="0 0 0"/>
+      <geometry>
+        <box size="${total_lenght} ${total_width} 0"/>
+      </geometry>
+      <material name="invisible_grey"/>
+    </visual>
+    <collision>
+      <origin rpy="0 0 0" xyz="0 0 0"/>
+      <geometry>
+        <box size="${total_lenght} ${total_width} 0"/>
+      </geometry>
+    </collision>
+  </link>
+  <joint name="base_link_to_base_footprint" type="fixed">
+    <origin xyz="0 0 0" rpy="0 0 0"/>
+    <parent link="base_link"/>
+    <child link="base_footprint"/>
+  </joint>
   <!-- chassis/body -->
   <joint name="base_link_to_link_chassis" type="fixed">

Commit message: [Description] - update description for D435

File: slammer_description/urdf/m2wr.xacro (robot description, xacro)
@@ -27,5 +27,5 @@
   <xacro:property name="camera_y_displacement" value="0.0"/>
   <xacro:property name="camera_z_displacement" value="0.07"/>
-  <xacro:property name="camera_rpy" value="0 0.22 0"/>
+  <xacro:property name="camera_rpy" value="0 0 0"/>
   <xacro:include filename="$(find slammer_description)/urdf/materials.xacro" />
   <xacro:include filename="$(find slammer_description)/urdf/m2wr.gazebo" />
