Commit message: Fix description(new imu orientation, joints), remove battery monitor (now integrated in uNav2)

File: slammer_description/urdf/macros.xacro (robot description, xacro)
@@ -24,5 +24,5 @@
   </xacro:macro>
   <xacro:macro name="joint_static_wheel" params="name child origin_xyz">
-    <joint name="${name}" type="fixed">
+    <joint name="${name}" type="continuous">
       <origin rpy="0 0 0" xyz="${origin_xyz}"/>
       <child link="${child}"/>
@@ -34,5 +34,5 @@
   </xacro:macro>
   <xacro:macro name="joint_wheel" params="name child origin_xyz">
-    <joint name="${name}" type="fixed">
+    <joint name="${name}" type="continuous">
       <origin rpy="0 0 0" xyz="${origin_xyz}"/>
       <child link="${child}"/>

File: slammer_description/urdf/slammer.xacro (robot description, xacro)
@@ -23,5 +23,5 @@
   <xacro:property name="imu_y_displacement" value="-0.05"/>
   <xacro:property name="imu_z_displacement" value="0.055"/>
-  <xacro:property name="imu_rpy" value="0 0.0 0"/>
+  <xacro:property name="imu_rpy" value="0 0 ${pi}"/>
   <xacro:property name="camera_x_displacement" value="0.145"/>
   <xacro:property name="camera_y_displacement" value="0.0"/>

Commit message: feat: update description, control configuration, teleop configuration

File: slammer_description/urdf/macros.xacro (robot description, xacro)
@@ -1,6 +1,6 @@
 <?xml version="1.0"?>
 <robot xmlns:xacro="http://www.ros.org/wiki/xacro">
-  <xacro:macro name="link_wheel" params="name">
-    <link name="${name}">
+<xacro:macro name="joint_wheel" params="name child origin_xyz">
+    <link name="${child}">
       <inertial>
         <mass value="0.2"/>
@@ -8,5 +8,5 @@
         <inertia ixx="0.000526666666667" ixy="0" ixz="0" iyy="0.000526666666667" iyz="0" izz="0.001"/>
       </inertial>
-      <collision name="${name}_collision">
+      <collision name="${child}_collision">
         <origin rpy="0 1.5707 1.5707" xyz="0 0 0"/>
         <geometry>
@@ -14,5 +14,5 @@
         </geometry>
       </collision>
-      <visual name="${name}_visual">
+      <visual name="${child}_visual">
         <origin rpy="0 1.5707 1.5707" xyz="0 0 0"/>
         <geometry>
@@ -22,24 +22,21 @@
       </visual>
     </link>
-  </xacro:macro>
-  <xacro:macro name="joint_static_wheel" params="name child origin_xyz">
     <joint name="${name}" type="continuous">
       <origin rpy="0 0 0" xyz="${origin_xyz}"/>
       <child link="${child}"/>
       <parent link="link_chassis"/>
-      <!-- <axis rpy="0 0 0" xyz="0 1 0"/>
-      <limit effort="10000" velocity="1000"/>
-      <joint_properties damping="1.0" friction="1.0"/ -->
-    </joint>
-  </xacro:macro>
-  <xacro:macro name="joint_wheel" params="name child origin_xyz">
-    <joint name="${name}" type="continuous">
-      <origin rpy="0 0 0" xyz="${origin_xyz}"/>
-      <child link="${child}"/>
-      <parent link="link_chassis"/>
-      <axis rpy="0 0 0" xyz="0 1 0"/>
+      <axis xyz="0 1 0"/>
       <limit effort="10000" velocity="1000"/>
       <joint_properties damping="1.0" friction="1.0"/>
     </joint>
+    <transmission name="${name}_transmission">
+      <type>transmission_interface/SimpleTransmission</type>
+      <joint name="${name}">
+        <hardwareInterface>hardware_interface/VelocityJointInterface</hardwareInterface>
+      </joint>
+      <actuator name="${name}_actuator">
+        <mechanicalReduction>1</mechanicalReduction>
+      </actuator>
+    </transmission>
   </xacro:macro>
   <xacro:macro name="cylinder_inertia" params="mass r l">

File: slammer_description/urdf/slammer.xacro (robot description, xacro)
@@ -122,12 +122,8 @@
   </link>
   <!-- Wheels -->
-  <xacro:link_wheel name="link_right_wheel" />
   <xacro:joint_wheel name="joint1" child="link_right_wheel" origin_xyz="${wheel_front_x_displacement} ${wheel_y_displacement} ${wheel_z_displacement}" />
-  <xacro:link_wheel name="link_left_wheel" />
   <xacro:joint_wheel name="joint2" child="link_left_wheel" origin_xyz="${wheel_front_x_displacement} ${-wheel_y_displacement} ${wheel_z_displacement}" />
-  <xacro:link_wheel name="link_rear_right_wheel" />
-  <xacro:joint_static_wheel name="joint3" child="link_rear_right_wheel" origin_xyz="${wheel_rear_x_displacement} ${wheel_y_displacement} ${wheel_z_displacement}" />
-  <xacro:link_wheel name="link_rear_left_wheel" />
-  <xacro:joint_static_wheel name="joint4" child="link_rear_left_wheel" origin_xyz="${wheel_rear_x_displacement} ${-wheel_y_displacement} ${wheel_z_displacement}" />
+  <xacro:joint_wheel name="joint3" child="link_rear_right_wheel" origin_xyz="${wheel_rear_x_displacement} ${wheel_y_displacement} ${wheel_z_displacement}" />
+  <xacro:joint_wheel name="joint4" child="link_rear_left_wheel" origin_xyz="${wheel_rear_x_displacement} ${-wheel_y_displacement} ${wheel_z_displacement}" />
   <!-- IMU -->
   <joint name="link_chassis_to_imu_bosch" type="fixed">

Commit message: fix ros control and description configuration

File: slammer_description/urdf/macros.xacro (robot description, xacro)
@@ -1,5 +1,5 @@
 <?xml version="1.0"?>
 <robot xmlns:xacro="http://www.ros.org/wiki/xacro">
-<xacro:macro name="joint_wheel" params="name child origin_xyz">
+<xacro:macro name="joint_wheel" params="name child origin_xyz axis">
     <link name="${child}">
       <inertial>
@@ -26,5 +26,5 @@
       <child link="${child}"/>
       <parent link="link_chassis"/>
-      <axis xyz="0 1 0"/>
+      <axis xyz="${axis}"/>
       <limit effort="10000" velocity="1000"/>
       <joint_properties damping="1.0" friction="1.0"/>

File: slammer_description/urdf/slammer.xacro (robot description, xacro)
@@ -122,8 +122,8 @@
   </link>
   <!-- Wheels -->
-  <xacro:joint_wheel name="joint1" child="link_right_wheel" origin_xyz="${wheel_front_x_displacement} ${wheel_y_displacement} ${wheel_z_displacement}" />
-  <xacro:joint_wheel name="joint2" child="link_left_wheel" origin_xyz="${wheel_front_x_displacement} ${-wheel_y_displacement} ${wheel_z_displacement}" />
-  <xacro:joint_wheel name="joint3" child="link_rear_right_wheel" origin_xyz="${wheel_rear_x_displacement} ${wheel_y_displacement} ${wheel_z_displacement}" />
-  <xacro:joint_wheel name="joint4" child="link_rear_left_wheel" origin_xyz="${wheel_rear_x_displacement} ${-wheel_y_displacement} ${wheel_z_displacement}" />
+  <xacro:joint_wheel name="joint1" child="link_right_wheel" origin_xyz="${wheel_front_x_displacement} ${-wheel_y_displacement} ${wheel_z_displacement}" axis="0 -1 0" />
+  <xacro:joint_wheel name="joint2" child="link_left_wheel" origin_xyz="${wheel_front_x_displacement} ${wheel_y_displacement} ${wheel_z_displacement}" axis="0 -1 0"/>
+  <xacro:joint_wheel name="joint3" child="link_rear_right_wheel" origin_xyz="${wheel_rear_x_displacement} ${-wheel_y_displacement} ${wheel_z_displacement}" axis="0 -1 0"/>
+  <xacro:joint_wheel name="joint4" child="link_rear_left_wheel" origin_xyz="${wheel_rear_x_displacement} ${wheel_y_displacement} ${wheel_z_displacement}" axis="0 -1 0"/>
   <!-- IMU -->
   <joint name="link_chassis_to_imu_bosch" type="fixed">

Commit message: fix: #2 motion sim working - todo: add odom noise

File: slammer_description/urdf/macros.xacro (robot description, xacro)
@@ -11,5 +11,5 @@
         <origin rpy="0 1.5707 1.5707" xyz="0 0 0"/>
         <geometry>
-          <cylinder length="0.065" radius="0.06"/>
+          <cylinder length="0.015" radius="0.06"/>
         </geometry>
       </collision>
@@ -17,5 +17,5 @@
         <origin rpy="0 1.5707 1.5707" xyz="0 0 0"/>
         <geometry>
-          <cylinder length="0.065" radius="0.06"/>
+          <cylinder length="0.015" radius="0.06"/>
         </geometry>
         <material name="black" />
